File: Kicad/Weather_station_unit/Weather_station_unit.kicad_pcb (KiCad board)
At the start: 2 copper layers, 0 parts

Commit message: final components routing for version 0.2
Parts:
- added BT1: BATTERY, custom:BATT_CONN, F.Cu at (143.4, 91.7)
- added C1: 1uF, Capacitors_SMD:C_0402, F.Cu at (147.7, 92.8)
- added C2: 100nF, Capacitors_SMD:C_0402, F.Cu at (163.7, 100.5)
- added C3: 10uF, Capacitors_SMD:C_0402, F.Cu at (163.7, 99.2)
- added C4: 100nF, Capacitors_SMD:C_0402, F.Cu at (163.7, 103.0)
- added C5: 1uF, Capacitors_SMD:C_0402, F.Cu at (147.8, 99.7)
- added C6: 0.1uF, Capacitors_SMD:C_0402, F.Cu at (154.2, 103.1)
- added C7: 0.1uF, Capacitors_SMD:C_0402, F.Cu at (161.7, 89.2)
- added C8: 0.1uF, Capacitors_SMD:C_0402, F.Cu at (152.4, 103.6)
- added C9: 0.1uF, Capacitors_SMD:C_0402, F.Cu at (154.9, 94.7)
- added D1: LED, custom:SMD-0402_LED, F.Cu at (147.8, 104.0)
- added D2: LED, custom:SMD-0402_LED, F.Cu at (166.9, 102.5)
- added IC1: ATMEGA328P-MM, custom:QFN-28-4x4mm_fixed_mask, F.Cu at (153.9, 98.8)
- added P1: FTDI CONN, custom:FTDI_PORT, F.Cu at (152.3, 89.1)
- added Q1: Oscilator, custom:ceramic_resonator_smd, F.Cu at (152.9, 94.5)
- added R1: PhotoResistor, Socket_Strips:Socket_Strip_Straight_1x02, F.Cu at (143.4, 101.2)
- added R2: 10K, Resistors_SMD:R_0402, F.Cu at (143.4, 106.5)
- added R3: 5K, Resistors_SMD:R_0402, F.Cu at (161.4, 106.0)
- added R4: 470, Resistors_SMD:R_0402, F.Cu at (147.8, 102.0)
- added R5: 10K, Resistors_SMD:R_0402, F.Cu at (168.0, 89.8)
- added R6: 4.7K, Resistors_SMD:R_0402, F.Cu at (164.9, 91.4)
- added R7: 10K, Resistors_SMD:R_0402, F.Cu at (168.0, 91.7)
- added R8: 4.7K, Resistors_SMD:R_0402, F.Cu at (164.9, 92.5)
- added R9: 470, Resistors_SMD:R_0402, F.Cu at (166.8, 100.5)
- added SW1: SW_PUSH, custom:push_switch_SMD, F.Cu at (181.1, 90.4)
- added TP1: TP1, custom:TEST_POINT, F.Cu at (145.2, 90.4)
- added TP10: TP10, custom:TEST_POINT, F.Cu at (155.1, 92.2)
- added TP2: TP2, custom:TEST_POINT, F.Cu at (155.6, 106.2)
- added TP3: Test_Point, custom:TEST_POINT, F.Cu at (150.1, 98.7)
- added TP4: TP4, custom:TEST_POINT, F.Cu at (163.9, 106.1)
- added TP5: TP5, custom:TEST_POINT, F.Cu at (170.3, 88.8)
- added TP6: TP6, custom:TEST_POINT, F.Cu at (177.8, 103.7)
- added TP7: TP7, custom:TEST_POINT, F.Cu at (171.4, 110.1)
- added TP8: TP8, custom:TEST_POINT, F.Cu at (156.1, 92.7)
- added TP9: TP9, custom:TEST_POINT, F.Cu at (170.7, 108.1)
- added U1: MPL3115A2, custom:MPL3115A2, F.Cu at (161.2, 99.3)
- added U2: MCP1802, custom:MCP1802T, F.Cu at (148.6, 95.0)
- added U3: DHT11, custom:DHT11, F.Cu at (166.0, 108.0)
- added U4: ESP-07, custom:ESP-07, F.Cu at (189.2, 110.1)
- added U5: ESP-01, custom:ESP-01, F.Cu at (180.0, 104.0)
- added conn1: I2C_CONN, custom:I2C_CONN, F.Cu at (165.4, 94.4)
- added conn2: SPI_CONN, custom:SPI_CONN, F.Cu at (152.1, 108.0)
Routing:
- net 3V3: track 0.00 -> 126.7 mm, vias 0 -> 1
- net GND: track 0.00 -> 46.2 mm, vias 0 -> 17
- net /TXS: track 0.00 -> 41.0 mm, vias 0 -> 4
- net /RXS: track 0.00 -> 40.6 mm, vias 0 -> 4
- net Net-(R7-Pad2): track 0.00 -> 33.2 mm, vias 0 -> 3
- net Net-(C7-Pad2): track 0.00 -> 31.6 mm
- net /SCK: track 0.00 -> 22.6 mm, vias 0 -> 2
- net /VCC: track 0.00 -> 21.4 mm
- net /D2: track 0.00 -> 17.9 mm, vias 0 -> 2
- net SDA: track 0.00 -> 16.0 mm, vias 0 -> 2
- net A0: track 0.00 -> 15.9 mm, vias 0 -> 1
- net /RX: track 0.00 -> 13.5 mm
- net SCL: track 0.00 -> 12.9 mm
- net /MISO: track 0.00 -> 11.4 mm, vias 0 -> 2
- net /TX: track 0.00 -> 11.4 mm, vias 0 -> 1
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- added copper zone on B.Cu, net GND
- added copper zone on F.Cu, net GND
Other:
- board outline added: 50.5 x 25.4 mm
- net class Default: clearance 0.254 -> 0.1524
- rule pad_to_mask_clearance: 0 -> 0.0508
- rule trace_clearance: 0.254 -> 0.1524
- rule trace_min: 0.254 -> 0.1524
- rule via_min_drill: 0.508 -> 0.3302
- rule via_min_size: 0.889 -> 0.508
- board text added: "Weather Spot Team"
- board text added: "Weather Station V.0.2"
